Commit message: finish the URDF integration, modified the readme a bit

File: ur_robotiq_description/urdf/ur.urdf.xacro (robot description, xacro)
@@ -30,4 +30,5 @@
    <xacro:arg name="trajectory_port" default="50003"/>
    <!--   tool communication related parameters-->
+   <xacro:arg name="tool_choice" default="none" />
    <xacro:arg name="use_tool_communication" default="false" />
    <xacro:arg name="tool_voltage" default="0" />
@@ -70,4 +71,5 @@
      headless_mode="$(arg headless_mode)"
      initial_positions="${xacro.load_yaml(initial_positions_file)}"
+     tool_choice="$(arg tool_choice)"
      use_tool_communication="$(arg use_tool_communication)"
      tool_voltage="$(arg tool_voltage)"

File: ur_robotiq_description/urdf/ur_macro.xacro (robot description, xacro)
@@ -65,4 +65,5 @@
     headless_mode:=false
     initial_positions:=${dict(shoulder_pan_joint=0.0,shoulder_lift_joint=-1.57,elbow_joint=0.0,wrist_1_joint=-1.57,wrist_2_joint=0.0,wrist_3_joint=0.0)}
+    tool_choice:=none
     use_tool_communication:=false
     tool_voltage:=0
@@ -378,8 +379,10 @@
       <child link="${tf_prefix}tool0"/>
     </joint>
-    <!-- <link name="${tf_prefix}gripper"/> -->
-    <xacro:robotiq_gripper name="RobotiqGripperHardwareInterface" prefix="" parent="${tf_prefix}tool0">
-      <origin xyz="0 0 0" rpy="0 0 0" />
-    </xacro:robotiq_gripper>
+    <!-- add gripper if requested -->
+    <xacro:if value="${tool_choice == 'robotiq_2f_85'}">
+      <xacro:robotiq_gripper name="RobotiqGripperHardwareInterface" prefix="" parent="${tf_prefix}tool0">
+        <origin xyz="0 0 0" rpy="0 0 0" />
+      </xacro:robotiq_gripper>
+    </xacro:if>
   </xacro:macro>
 </robot>
