Commit message: add moveit configuration. Although I am doubting its usefulness. Need some testing

File: ur_robotiq_description/urdf/2f_85/robotiq_2f_85_macro.urdf.xacro (robot description, xacro)
@@ -15,5 +15,5 @@
         com_port:=/dev/ttyUSB0">
         <!-- ros2 control include -->
-        <xacro:include filename="$(find robotiq_description)/urdf/2f_85.ros2_control.xacro" />
+        <xacro:include filename="$(find ur_robotiq_description)/urdf/2f_85/2f_85.ros2_control.xacro" />
         <!-- if we are simulating or directly communicating with the gripper we need a ros2 control instance -->
         <xacro:if value="${include_ros2_control}">
@@ -31,10 +31,10 @@
             <visual>
                 <geometry>
-                    <mesh filename="file://$(find robotiq_description)/meshes/visual/2f_85/robotiq_base.dae" />
-                </geometry>
-            </visual>
-            <collision>
-                <geometry>
-                    <mesh filename="file://$(find robotiq_description)/meshes/collision/2f_85/robotiq_base.stl" />
+                    <mesh filename="file://$(find ur_robotiq_description)/meshes/2f_85/visual/robotiq_base.dae" />
+                </geometry>
+            </visual>
+            <collision>
+                <geometry>
+                    <mesh filename="file://$(find ur_robotiq_description)/meshes/2f_85/collision/robotiq_base.stl" />
                 </geometry>
             </collision>
@@ -48,10 +48,10 @@
             <visual>
                 <geometry>
-                    <mesh filename="file://$(find robotiq_description)/meshes/visual/2f_85/left_knuckle.dae" />
-                </geometry>
-            </visual>
-            <collision>
-                <geometry>
-                    <mesh filename="file://$(find robotiq_description)/meshes/collision/2f_85/left_knuckle.stl" />
+                    <mesh filename="file://$(find ur_robotiq_description)/meshes/2f_85/visual/left_knuckle.dae" />
+                </geometry>
+            </visual>
+            <collision>
+                <geometry>
+                    <mesh filename="file://$(find ur_robotiq_description)/meshes/2f_85/collision/left_knuckle.stl" />
                 </geometry>
             </collision>
@@ -65,10 +65,10 @@
             <visual>
                 <geometry>
-                    <mesh filename="file://$(find robotiq_description)/meshes/visual/2f_85/right_knuckle.dae" />
-                </geometry>
-            </visual>
-            <collision>
-                <geometry>
-                    <mesh filename="file://$(find robotiq_description)/meshes/collision/2f_85/right_knuckle.stl" />
+                    <mesh filename="file://$(find ur_robotiq_description)/meshes/2f_85/visual/right_knuckle.dae" />
+                </geometry>
+            </visual>
+            <collision>
+                <geometry>
+                    <mesh filename="file://$(find ur_robotiq_description)/meshes/2f_85/collision/right_knuckle.stl" />
                 </geometry>
             </collision>
@@ -82,10 +82,10 @@
             <visual>
                 <geometry>
-                    <mesh filename="file://$(find robotiq_description)/meshes/visual/2f_85/left_finger.dae" />
-                </geometry>
-            </visual>
-            <collision>
-                <geometry>
-                    <mesh filename="file://$(find robotiq_description)/meshes/collision/2f_85/left_finger.stl" />
+                    <mesh filename="file://$(find ur_robotiq_description)/meshes/2f_85/visual/left_finger.dae" />
+                </geometry>
+            </visual>
+            <collision>
+                <geometry>
+                    <mesh filename="file://$(find ur_robotiq_description)/meshes/2f_85/collision/left_finger.stl" />
                 </geometry>
             </collision>
@@ -99,10 +99,10 @@
             <visual>
                 <geometry>
-                    <mesh filename="file://$(find robotiq_description)/meshes/visual/2f_85/right_finger.dae" />
-                </geometry>
-            </visual>
-            <collision>
-                <geometry>
-                    <mesh filename="file://$(find robotiq_description)/meshes/collision/2f_85/right_finger.stl" />
+                    <mesh filename="file://$(find ur_robotiq_description)/meshes/2f_85/visual/right_finger.dae" />
+                </geometry>
+            </visual>
+            <collision>
+                <geometry>
+                    <mesh filename="file://$(find ur_robotiq_description)/meshes/2f_85/collision/right_finger.stl" />
                 </geometry>
             </collision>
@@ -116,10 +116,10 @@
             <visual>
                 <geometry>
-                    <mesh filename="file://$(find robotiq_description)/meshes/visual/2f_85/left_inner_knuckle.dae" />
-                </geometry>
-            </visual>
-            <collision>
-                <geometry>
-                    <mesh filename="file://$(find robotiq_description)/meshes/collision/2f_85/left_inner_knuckle.stl" />
+                    <mesh filename="file://$(find ur_robotiq_description)/meshes/2f_85/visual/left_inner_knuckle.dae" />
+                </geometry>
+            </visual>
+            <collision>
+                <geometry>
+                    <mesh filename="file://$(find ur_robotiq_description)/meshes/2f_85/collision/left_inner_knuckle.stl" />
                 </geometry>
             </collision>
@@ -133,10 +133,10 @@
             <visual>
                 <geometry>
-                    <mesh filename="file://$(find robotiq_description)/meshes/visual/2f_85/right_inner_knuckle.dae" />
-                </geometry>
-            </visual>
-            <collision>
-                <geometry>
-                    <mesh filename="file://$(find robotiq_description)/meshes/collision/2f_85/right_inner_knuckle.stl" />
+                    <mesh filename="file://$(find ur_robotiq_description)/meshes/2f_85/visual/right_inner_knuckle.dae" />
+                </geometry>
+            </visual>
+            <collision>
+                <geometry>
+                    <mesh filename="file://$(find ur_robotiq_description)/meshes/2f_85/collision/right_inner_knuckle.stl" />
                 </geometry>
             </collision>
@@ -150,10 +150,10 @@
             <visual>
                 <geometry>
-                    <mesh filename="file://$(find robotiq_description)/meshes/visual/2f_85/left_finger_tip.dae" />
-                </geometry>
-            </visual>
-            <collision>
-                <geometry>
-                    <mesh filename="file://$(find robotiq_description)/meshes/collision/2f_85/left_finger_tip.stl" />
+                    <mesh filename="file://$(find ur_robotiq_description)/meshes/2f_85/visual/left_finger_tip.dae" />
+                </geometry>
+            </visual>
+            <collision>
+                <geometry>
+                    <mesh filename="file://$(find ur_robotiq_description)/meshes/2f_85/collision/left_finger_tip.stl" />
                 </geometry>
                 <surface>
@@ -185,10 +185,10 @@
             <visual>
                 <geometry>
-                    <mesh filename="file://$(find robotiq_description)/meshes/visual/2f_85/right_finger_tip.dae" />
-                </geometry>
-            </visual>
-            <collision>
-                <geometry>
-                    <mesh filename="file://$(find robotiq_description)/meshes/collision/2f_85/right_finger_tip.stl" />
+                    <mesh filename="file://$(find ur_robotiq_description)/meshes/2f_85/visual/right_finger_tip.dae" />
+                </geometry>
+            </visual>
+            <collision>
+                <geometry>
+                    <mesh filename="file://$(find ur_robotiq_description)/meshes/2f_85/collision/right_finger_tip.stl" />
                 </geometry>
                 <surface>
